File: bGeigie3.brd (EAGLE design)
At the start: 80 x 80 mm, 106 parts, among them Q1 FDN360P, Q2 16MHz, Q3 8MHz, Q4 8MHz, Q5 FDN360P, Q6 FDN360P, Q7 FDN360P

Commit message: Added serial header for debugging.
Parts:
- added SERIAL1: (no value), pinhead:1X04
Connections:
- net GND: now also SERIAL1.4
- net RX0: now also SERIAL1.3
- net TX0: now also SERIAL1.2
- net VCC3: now also SERIAL1.1
Routing:
- net RX0: track 37.6 -> 62.7 mm
- net TX0: track 42.1 -> 66.2 mm
- net VCC3: track 346.6 -> 363.9 mm
- net RESET: track 189.6 -> 203.8 mm, vias 12 -> 14
- net GND: vias 195 -> 187
Other:
- board text added: "3.3V"
- board text added: "GND"
- board text added: "RX"
- board text added: "TX"
- board text added: "bGeigie v3.6"
- board text removed: "bGeigie v3.5"
Changed lines of the file:
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@@
 <text x="16.5354" y="43.2308" size="0.8128" layer="22" rot="MR0">Charging</text>
 <text x="16.51" y="40.894" size="0.8128" layer="22" rot="MR0">USB</text>
-<text x="54.991" y="0.7874" size="1.778" layer="21" ratio="10">bGeigie v3.5</text>
+<text x="54.991" y="0.7874" size="1.778" layer="21" ratio="10">bGeigie v3.6</text>
 <text x="39.5732" y="20.9042" size="1.27" layer="21">by FakuFaku</text>
 <text x="39.5224" y="19.2024" size="1.27" layer="21">November 2013</text>
@@
 <text x="22.5044" y="41.9608" size="0.508" layer="26" rot="MR0">LED2_BK</text>
 <text x="22.5552" y="40.7416" size="0.508" layer="26" rot="MR0">LED3_BK</text>
+<text x="76.5556" y="34.7472" size="1.016" layer="25" rot="R180">3.3V</text>
+<text x="76.5556" y="29.718" size="1.016" layer="25" rot="R180">RX</text>
+<text x="76.5556" y="32.2072" size="1.016" layer="25" rot="R180">TX</text>
+<text x="76.5556" y="27.1272" size="1.016" layer="25" rot="R180">GND</text>
 </plain>
 <attributes>
@@
 </element>
 <element name="C37" library="Robin" package="D/7343-31W" value="" x="27.8384" y="48.3108" rot="R90"/>
+<element name="SERIAL1" library="pinhead" package="1X04" value="" x="78.0796" y="30.4292" smashed="yes" rot="R270">
+<attribute name="VALUE" x="74.9046" y="35.5092" size="1.27" layer="27" rot="R270"/>
+</element>
 </elements>
 <signals>
@@
 <via x="60.96" y="60.9092" extent="1-16" drill="0.3048"/>
 <via x="60.96" y="50.8508" extent="1-16" drill="0.3048"/>
-<via x="77.8256" y="31.3944" extent="1-16" drill="0.3048"/>
-<via x="77.6224" y="33.8836" extent="1-16" drill="0.3048"/>
-<via x="77.6224" y="28.702" extent="1-16" drill="0.3048"/>
+<via x="78.1812" y="40.5384" extent="1-16" drill="0.3048"/>
 <via x="62.5348" y="3.2512" extent="1-16" drill="0.3048"/>
 <via x="11.3792" y="70.9168" extent="1-16" drill="0.3048"/>
@@
 <via x="64.7192" y="17.8308" extent="1-16" drill="0.3048"/>
 <via x="75.1332" y="18.3896" extent="1-16" drill="0.3048"/>
-<via x="73.3044" y="24.5364" extent="1-16" drill="0.3048"/>
+<via x="73.2536" y="24.638" extent="1-16" drill="0.3048"/>
 <via x="78.3336" y="18.3896" extent="1-16" drill="0.3048"/>
 <via x="78.3336" y="20.2692" extent="1-16" drill="0.3048"/>
@@
 <via x="10.2616" y="5.7912" extent="1-16" drill="0.3048"/>
 <via x="10.2616" y="2.9972" extent="1-16" drill="0.3048"/>
-<via x="74.4728" y="23.0124" extent="1-16" drill="0.3048"/>
-<via x="76.4032" y="22.9616" extent="1-16" drill="0.3048"/>
-<via x="70.3072" y="34.7472" extent="1-16" drill="0.3048"/>
+<via x="78.6384" y="22.8092" extent="1-16" drill="0.3048"/>
+<via x="70.358" y="36.2712" extent="1-16" drill="0.3048"/>
 <via x="68.8848" y="36.322" extent="1-16" drill="0.3048"/>
 <via x="71.882" y="36.2712" extent="1-16" drill="0.3048"/>
@@
 <vertex x="46.736" y="9.0932"/>
 </polygon>
-<via x="56.7944" y="30.6324" extent="1-16" drill="0.3048"/>
-<via x="58.6232" y="30.6324" extent="1-16" drill="0.3048"/>
 <via x="57.7088" y="26.5684" extent="1-16" drill="0.3048"/>
 <via x="57.7088" y="27.686" extent="1-16" drill="0.3048"/>
-<via x="57.6072" y="30.6324" extent="1-16" drill="0.3048"/>
 <via x="61.6204" y="24.5872" extent="1-16" drill="0.3048"/>
 <via x="57.3532" y="33.6296" extent="1-16" drill="0.3048"/>
@@
 <via x="75.8952" y="50.546" extent="1-16" drill="0.3048"/>
 <via x="75.8952" y="54.0512" extent="1-16" drill="0.3048"/>
-<via x="75.9968" y="34.8488" extent="1-16" drill="0.3048"/>
-<via x="75.692" y="31.5976" extent="1-16" drill="0.3048"/>
-<via x="75.3364" y="27.3812" extent="1-16" drill="0.3048"/>
+<via x="78.0796" y="42.418" extent="1-16" drill="0.3048"/>
 <via x="77.7748" y="44.9072" extent="1-16" drill="0.3048"/>
-<via x="73.7108" y="46.99" extent="1-16" drill="0.3048"/>
 <via x="77.978" y="50.546" extent="1-16" drill="0.3048"/>
 <via x="73.8124" y="54.0512" extent="1-16" drill="0.3048"/>
+<contactref element="SERIAL1" pad="4"/>
+<via x="69.2404" y="21.2344" extent="1-16" drill="0.3048"/>
 </signal>
 <signal name="VBUS">
@@
 <wire x1="72.5424" y1="18.7452" x2="72.5424" y2="19.5462" width="0.762" layer="1"/>
 <wire x1="72.5424" y1="19.5462" x2="72.5796" y2="19.5834" width="0.762" layer="1"/>
+<contactref element="SERIAL1" pad="1"/>
+<wire x1="72.6288" y1="21.6584" x2="74.084" y2="21.6584" width="0.762" layer="1"/>
+<wire x1="74.084" y1="21.6584" x2="74.7776" y2="22.352" width="0.762" layer="1"/>
+<wire x1="74.7776" y1="22.352" x2="74.7776" y2="33.6804" width="0.762" layer="1"/>
+<wire x1="74.7776" y1="33.6804" x2="75.3364" y2="34.2392" width="0.762" layer="1"/>
+<wire x1="75.3364" y1="34.2392" x2="78.0796" y2="34.2392" width="0.762" layer="1"/>
 </signal>
 <signal name="RESET">
@@
 <via x="55.2196" y="12.5984" extent="1-16" drill="0.3048"/>
 <wire x1="55.2196" y1="12.5984" x2="61.9252" y2="19.304" width="0.3048" layer="16"/>
-<wire x1="61.9252" y1="19.304" x2="63.3476" y2="19.304" width="0.3048" layer="16"/>
-<wire x1="63.3476" y1="19.304" x2="64.5668" y2="20.5232" width="0.3048" layer="16"/>
-<wire x1="64.5668" y1="20.5232" x2="64.5668" y2="21.5392" width="0.3048" layer="16"/>
-<wire x1="64.5668" y1="21.5392" x2="64.0588" y2="22.0472" width="0.3048" layer="16"/>
-<wire x1="64.0588" y1="22.0472" x2="64.0588" y2="29.4132" width="0.3048" layer="16"/>
-<wire x1="64.0588" y1="29.4132" x2="61.5696" y2="31.9024" width="0.3048" layer="16"/>
-<wire x1="61.5696" y1="31.9024" x2="61.5696" y2="35.052" width="0.3048" layer="16"/>
-<wire x1="61.5696" y1="35.052" x2="61.0108" y2="35.6108" width="0.3048" layer="16"/>
+<wire x1="61.6712" y1="34.9504" x2="61.0108" y2="35.6108" width="0.3048" layer="16"/>
+<wire x1="61.9252" y1="19.304" x2="64.9224" y2="19.304" width="0.3048" layer="16"/>
+<wire x1="64.9224" y1="19.304" x2="72.9996" y2="27.3812" width="0.3048" layer="16"/>
+<wire x1="72.9996" y1="27.3812" x2="72.9996" y2="28.1432" width="0.3048" layer="16"/>
+<via x="72.9996" y="28.1432" extent="1-16" drill="0.3048"/>
+<wire x1="72.9996" y1="28.1432" x2="72.9996" y2="34.3916" width="0.3048" layer="1"/>
+<wire x1="72.9996" y1="34.3916" x2="72.4408" y2="34.9504" width="0.3048" layer="1"/>
+<via x="72.4408" y="34.9504" extent="1-16" drill="0.3048"/>
+<wire x1="72.4408" y1="34.9504" x2="61.6712" y2="34.9504" width="0.3048" layer="16"/>
 </signal>
 <signal name="N$6">
@@
 <wire x1="50.0292" y1="27.0386" x2="52.9466" y2="27.0386" width="0.4064" layer="1"/>
 <wire x1="52.9466" y1="27.0386" x2="53.2384" y2="27.3304" width="0.4064" layer="1"/>
+<contactref element="SERIAL1" pad="3"/>
+<wire x1="53.2384" y1="30.2768" x2="75.8952" y2="30.2768" width="0.4064" layer="16"/>
+<wire x1="75.8952" y1="30.2768" x2="78.0796" y2="29.1592" width="0.4064" layer="16"/>
 </signal>
 <signal name="TX0">
-<contactref element="1284P" pad="10"/>
-<wire x1="50.0292" y1="26.2386" x2="50.0542" y2="26.2636" width="0.3048" layer="1"/>
 <contactref element="32U4" pad="20"/>
 <wire x1="28.0576" y1="23.521" x2="28.0576" y2="31.1056" width="0.4064" layer="1"/>
@@
 <wire x1="54.102" y1="27.0256" x2="53.34" y2="26.2636" width="0.4064" layer="1"/>
 <wire x1="50.0542" y1="26.2636" x2="53.34" y2="26.2636" width="0.4064" layer="1"/>
+<contactref element="1284P" pad="10"/>
+<contactref element="SERIAL1" pad="2"/>
+<wire x1="54.102" y1="31.0896" x2="76.4032" y2="31.0896" width="0.4064" layer="16"/>
+<wire x1="76.4032" y1="31.0896" x2="78.0796" y2="31.6992" width="0.4064" layer="16"/>
+<wire x1="50.0542" y1="26.2636" x2="50.0292" y2="26.2386" width="0.3048" layer="1"/>
 </signal>
 <signal name="MOSI">
